File: HUD-eaglefiles/HUD.sch (EAGLE design)
At the start: 72 parts, among them U1 LM317, U2 ATMEGA328P_TQFP

Commit message: added display power output in the motherboard and created the display schematic file
Parts:
- added DIS_PWR_SELECT: JUMPER-3PTH, SparkFun-Retired:JUMPER-3PTH
- added PWR_PINS_OUT: (no value), SparkFun-Connectors:M02PTH
- added R27: (no value), SparkFun-Resistors:RESISTORPTH-1/4W
- renumbered Q1 to QA0, Q10 to QC1, Q11 to QD1, Q12 to QE1, Q13 to QF1, Q14 to QG1, Q15 to QA2, Q16 to QB2, Q17 to QC2, Q18 to QD2, Q19 to QE2, Q2 to QB0, Q20 to QF2, Q21 to QG2, Q3 to QC0, Q4 to QD0, Q5 to QE0, Q6 to QF0, Q7 to QG0, Q8 to QA1, Q9 to QB1
Connections:
- net N$19 renamed RESET_WIRE
- net N$3 renamed PWRIN
- new net 12VOUT: DIS_PWR_SELECT.3, R27.2
- new net DISPLAY_PWR-OUT: DIS_PWR_SELECT.2, PWR_PINS_OUT.1
- net GND: now also PWR_PINS_OUT.2
- net RAW: now also R27.1
- net VCC: now also DIS_PWR_SELECT.1
Other:
- note added: "Dosplay Power Out"

Commit message: renamed tranisitors and modified the arrangment, and added valuse for all components
Parts:
- removed JP5: (no value), SparkFun:M02PTH
- AOUT, DOUT: value (none) -> female_header
- AOUT_H, DOUT_H: value (none) -> holes
- COM_SERIAL, OBD_SERIAL: value (none) -> male_header
- D0_IN, D1_IN, D2_IN, PWR_PINS_OUT: value (none) -> DConnector
- JP1: value (none) -> Pwr_in
- R27: value (none) -> 1K
Connections:
- net GND: no longer JP5.2
- net PWRIN: no longer JP5.1
Other:
- note added: "Display Power Out"
- note removed: "Dosplay Power Out"
- moved on the sheet: DIS_PWR_SELECT, PWR_PINS_OUT, R27
